File: MCU.kicad_sch (KiCad schematic)
At the start: 38 parts, among them U1 SN74AHC1G02, U8 74VHC4053AFT

Commit message: Use kicad footprints for resistors/capacitors
Parts:
- C1, C2, C26, C29, C30, C32, C33: footprint 32blit:C0603 -> Capacitor_SMD:C_0603_1608Metric
- C11, C4, C5, C6, C7, C8, C9: footprint 32blit:C0402K -> Capacitor_SMD:C_0402_1005Metric
- C24, C35: footprint 32blit:C0603K -> Capacitor_SMD:C_0603_1608Metric
- R1, R13, R21, R29, R9: footprint 32blit:R0603 -> Resistor_SMD:R_0603_1608Metric

Commit message: More footprint replacements
This involved some adjusting for pad sizes
Parts:
- STM32H750: footprint 32blit:LQFP-100 -> Package_QFP:LQFP-100_14x14mm_P0.5mm
- U$17, U$22, U$23: footprint 32blit:FIDUCIAL-1MM -> Fiducial:Fiducial_1mm_Mask2mm
- U$19: footprint 32blit:TSX-3225 -> Crystal:Crystal_SMD_SeikoEpson_TSX3225-4Pin_3.2x2.5mm
- U1: footprint 32blit:SOT-23-5 -> Package_TO_SOT_SMD:SOT-23-5
- U8: footprint 32blit:TSSOP-16-TI -> Package_SO:TSSOP-16_4.4x5mm_P0.65mm
Changed lines of the file:
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@@
       (effects (font (size 1.27 1.27)) hide)
     )
-    (property "Footprint" "32blit:TSX-3225" (at 48.26 231.14 0)
+    (property "Footprint" "Crystal:Crystal_SMD_SeikoEpson_TSX3225-4Pin_3.2x2.5mm" (at 48.26 231.14 0)
       (effects (font (size 1.27 1.27)) hide)
     )
@@
       (effects (font (size 1.27 1.27)) hide)
     )
-    (property "Footprint" "32blit:FIDUCIAL-1MM" (at 297.18 274.32 0)
+    (property "Footprint" "Fiducial:Fiducial_1mm_Mask2mm" (at 297.18 274.32 0)
       (effects (font (size 1.27 1.27)) hide)
     )
@@
       (effects (font (size 1.27 1.27)) hide)
     )
-    (property "Footprint" "32blit:TSSOP-16-TI" (at 340.36 162.56 0)
+    (property "Footprint" "Package_SO:TSSOP-16_4.4x5mm_P0.65mm" (at 340.36 162.56 0)
       (effects (font (size 1.27 1.27)) hide)
     )
@@
       (effects (font (size 1.27 1.27)) hide)
     )
-    (property "Footprint" "32blit:LQFP-100" (at 119.38 149.86 0)
+    (property "Footprint" "Package_QFP:LQFP-100_14x14mm_P0.5mm" (at 119.38 149.86 0)
       (effects (font (size 1.27 1.27)) hide)
     )
@@
       (effects (font (size 1.27 1.27)) hide)
     )
-    (property "Footprint" "32blit:FIDUCIAL-1MM" (at 302.26 274.32 0)
+    (property "Footprint" "Fiducial:Fiducial_1mm_Mask2mm" (at 302.26 274.32 0)
       (effects (font (size 1.27 1.27)) hide)
     )
@@
       (effects (font (size 1.27 1.27)) hide)
     )
-    (property "Footprint" "32blit:SOT-23-5" (at 340.36 104.14 0)
+    (property "Footprint" "Package_TO_SOT_SMD:SOT-23-5" (at 340.36 104.14 0)
       (effects (font (size 1.27 1.27)) hide)
     )
@@
       (effects (font (size 1.27 1.27)) hide)
     )
-    (property "Footprint" "32blit:FIDUCIAL-1MM" (at 292.1 274.32 0)
-      (effects (font (size 1.27 1.27)) hide)
-    )
+    (property "Footprint" "Fiducial:Fiducial_1mm_Mask2mm" (at 292.1 274.32 0)
+      (effects (font (size 1.27 1.27)) hide)
+    )

Commit message: Remove custom pimoroni frame
Makes the sch a bit hard to work with and recreating it in the .kicad_wks seems difficult
Other:
- title: (none) -> 32blit
Changed lines of the file:
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@@
 (kicad_sch (version 20230121) (generator eeschema)
   (paper "User" 426.949 302.158)
+  (title_block
+    (title "32blit")
+  )
   (junction (at 53.34 134.62) (diameter 0) (color 0 0 0 0)
   )
@@
         )
       )
-    )
-  )
-  (symbol (lib_id "32blit-eagle-import:DINA3_PIM_L") (at 17.78 281.94 0) (unit 1)
-    (in_bom yes) (on_board yes) (dnp no)
-    (property "Reference" "#FRAME3" (at 17.78 281.94 0)
-      (effects (font (size 1.27 1.27)) hide)
-    )
-    (property "Value" "DINA3_PIM_L" (at 17.78 281.94 0)
-      (effects (font (size 1.27 1.27)) hide)
-    )
-    (property "Footprint" "" (at 17.78 281.94 0)
-      (effects (font (size 1.27 1.27)) hide)
-    )
-    (property "Datasheet" "" (at 17.78 281.94 0)
-      (effects (font (size 1.27 1.27)) hide)
-    )
-    (instances
-      (project "32blit"
-        (path "/5e392b0a-93d8-4fe3-995e-b41db5e69183/7029eee7-bbab-4242-813a-e587b6182828"
-          (reference "#FRAME3") (unit 1)
-        )
-      )

Commit message: Giant schematic rework
Use as many kicad symbols as possiblem, adjust remaining imported symbols to make ERC happy and adjust some footprints for the new symbols
Parts:
- C1, C2, C26, C29, C30, C32, C33: symbol 32blit-eagle-import:C-EUC0603 -> Device:C
- C11, C4, C5, C6, C7, C8, C9: symbol 32blit-eagle-import:rcl_C-EUC0402K -> Device:C
- C24, C35: symbol 32blit-eagle-import:rcl_C-EUC0603K -> Device:C
- JP1: symbol 32blit-eagle-import:10-WAY -> Connector_Generic:Conn_01x10
- R1, R13, R21, R29, R9: symbol 32blit-eagle-import:R-EU_R0603 -> Device:R
- STM32H750: symbol 32blit-eagle-import:STM32H750VB -> MCU_ST_STM32H7:STM32H750VBTx
- SWRESET0: symbol 32blit-eagle-import:TACT_SWITCHLOWPROFILE -> Switch:SW_Push
- U$17, U$22, U$23: symbol 32blit-eagle-import:FIDUCIAL1MM -> Mechanical:Fiducial
- U$19: symbol 32blit-eagle-import:TSX-3225 -> Device:Crystal_GND24
- U1: symbol 32blit-eagle-import:SN74AHC1G02 -> 74xGxx:74AHC1G02
- USER_3V3_1, USER_3V3_2, USER_GND_1, USER_GND_2, USER_LEFT1, USER_LEFT2, USER_RIGHT1, USER_RIGHT2: symbol 32blit-eagle-import:TPTP17SQ -> Connector:TestPoint_Alt
Connections:
- net BOOT0: now also JP1.10 (Pin_10); no longer JP1.A10 (10), JP1.B10 (10)
- net EXTENSION_GPIO: now also JP1.2 (Pin_2); no longer JP1.A2 (2), JP1.B2 (2)
- net GND: now also JP1.1 (Pin_1), JP1.7 (Pin_7), SWRESET0.2, USER_GND_1.1, USER_GND_2.1; no longer JP1.A1 (1), JP1.A7 (7), JP1.B1 (1), JP1.B7 (7), SWRESET0.3 (2), SWRESET0.4 (2), USER_GND_1.TP, USER_GND_2.TP
- net I2C_SCL: now also JP1.3 (Pin_3); no longer JP1.A3 (3), JP1.B3 (3)
- net I2C_SDA: now also JP1.4 (Pin_4); no longer JP1.A4 (4), JP1.B4 (4)
- net SWCLK: now also JP1.6 (Pin_6); no longer JP1.A6 (6), JP1.B6 (6)
- net SWDIO: now also JP1.8 (Pin_8); no longer JP1.A8 (8), JP1.B8 (8)
- net USER_LEFT1: now also USER_LEFT1.1; no longer USER_LEFT1.TP
- net USER_LEFT2: now also USER_LEFT2.1; no longer USER_LEFT2.TP
- net USER_RIGHT1: now also USER_RIGHT1.1; no longer USER_RIGHT1.TP
- net USER_RIGHT2: now also USER_RIGHT2.1; no longer USER_RIGHT2.TP
- net ~{RESET}: now also JP1.9 (Pin_9); no longer JP1.A9 (9), JP1.B9 (9), SWRESET0.2 (1)
- net at U$19.2: no longer U$19.4 (GND)
- net 3V3 renamed +3.3V
- net +3.3V: now also JP1.5 (Pin_5), USER_3V3_1.1, USER_3V3_2.1; no longer JP1.A5 (5), JP1.B5 (5), USER_3V3_1.TP, USER_3V3_2.TP
- net USB_5V renamed VBUS
- no-connect marks 0 -> 5
